Commit message: Added GPU option

File: arti_gazebo_ouster/urdf/OS1-16.urdf.xacro (robot description, xacro)
@@ -2,5 +2,5 @@
 <robot xmlns:xacro="http://ros.org/wiki/xacro" name="OS1-16">
   <xacro:property name="M_PI" value="3.1415926535897931" />
-  <xacro:macro name="OS1-16" params="*origin parent:=base_link name:=os1_sensor topic_points:=/os1_cloud_node/points topic_imu:=/os1_cloud_node/imu hz:=10 samples:=512 min_range:=0.9 max_range:=75.0 noise:=0.008 min_angle:=-${M_PI} max_angle:=${M_PI} lidar_link:=os1_lidar imu_link:=os1_imu vfov_min:=-.26 vfov_max:=.26">
+  <xacro:macro name="OS1-16" params="*origin parent:=base_link name:=os1_sensor topic_points:=/os1_cloud_node/points topic_imu:=/os1_cloud_node/imu hz:=10 samples:=512 min_range:=0.9 max_range:=75.0 noise:=0.008 min_angle:=-${M_PI} max_angle:=${M_PI} lidar_link:=os1_lidar imu_link:=os1_imu vfov_min:=-.29 vfov_max:=.29 gpu:=false">
     <joint name="${name}_mount_joint" type="fixed">
       <xacro:insert_block name="origin" />
@@ -43,5 +43,41 @@
     </joint>
     <!-- Gazebo requires the ouster_gazebo_plugins package -->
-    <gazebo reference="${name}">
+    <gazebo reference="${lidar_link}">
+      <xacro:if value="${gpu}">
+        <sensor type="gpu_ray" name="${name}-OS1-16">
+          <pose>0 0 0 0 0 0</pose>
+          <visualize>false</visualize>
+          <update_rate>${hz}</update_rate>
+          <ray>
+            <scan>
+              <horizontal>
+                <samples>${samples}</samples>
+                <resolution>1</resolution>
+                <min_angle>${min_angle}</min_angle>
+                <max_angle>${max_angle}</max_angle>
+              </horizontal>
+              <vertical>
+                <samples>16</samples>
+                <resolution>1</resolution>
+                <min_angle>${vfov_min}</min_angle>
+                <max_angle>${vfov_max}</max_angle>
+              </vertical>
+            </scan>
+            <range>
+              <min>${min_range}</min>
+              <max>${max_range}</max>
+              <resolution>0.03</resolution>
+            </range>
+          </ray>
+          <plugin name="gazebo_ros_laser_controller" filename="libgazebo_ros_ouster_gpu_laser.so">
+            <topicName>${topic_points}</topicName>
+            <frameName>${lidar_link}</frameName>
+            <min_range>${min_range}</min_range>
+            <max_range>${max_range}</max_range>
+            <gaussianNoise>${noise}</gaussianNoise>
+          </plugin>
+        </sensor>
+      </xacro:if>
+      <xacro:unless value="${gpu}">
         <sensor type="ray" name="${name}-OS1-16">
           <pose>0 0 0 0 0 0</pose>
@@ -77,4 +113,5 @@
           </plugin>
         </sensor>
+      </xacro:unless>
     </gazebo>
     <!-- IMU -->

Commit message: small modification

File: arti_gazebo_ouster/urdf/OS1-16.urdf.xacro (robot description, xacro)
@@ -22,5 +22,5 @@
       </collision>
       <visual name="base_visual">
-         <origin xyz="0 0 0.0" rpy="0 0 1.5707" />
+         <origin xyz="0 0 0.0365" rpy="0 0 1.5707" />
          <geometry>
 	         <mesh filename="package://arti_gazebo_ouster/meshes/os1_64.dae" />

File: arti_gazebo_ouster/urdf/OS1-32.urdf.xacro (robot description, xacro)
@@ -2,5 +2,5 @@
 <robot xmlns:xacro="http://ros.org/wiki/xacro" name="OS1-32">
   <xacro:property name="M_PI" value="3.1415926535897931" />
-  <xacro:macro name="OS1-32" params="*origin parent:=base_link name:=os1_sensor topic_points:=/os1_cloud_node/points topic_imu:=/os1_cloud_node/imu hz:=10 samples:=512 min_range:=0.9 max_range:=75.0 noise:=0.008 min_angle:=-${M_PI} max_angle:=${M_PI} lidar_link:=os1_lidar imu_link:=os1_imu vfov_min:=-.26 vfov_max:=.26">
+  <xacro:macro name="OS1-32" params="*origin parent:=base_link name:=os1_sensor topic_points:=/os1_cloud_node/points topic_imu:=/os1_cloud_node/imu hz:=10 samples:=512 min_range:=0.9 max_range:=75.0 noise:=0.008 min_angle:=-${M_PI} max_angle:=${M_PI} lidar_link:=os1_lidar imu_link:=os1_imu vfov_min:=-.26 vfov_max:=.26 gpu:=false">
     <joint name="${name}_mount_joint" type="fixed">
       <xacro:insert_block name="origin" />
@@ -22,5 +22,5 @@
       </collision>
       <visual name="base_visual">
-         <origin xyz="0 0 0.0" rpy="0 0 1.5707" />
+         <origin xyz="0 0 0.0365" rpy="0 0 1.5707" />
          <geometry>
 	         <mesh filename="package://arti_gazebo_ouster/meshes/os1_64.dae" />
@@ -43,5 +43,41 @@
     </joint>
     <!-- Gazebo requires the ouster_gazebo_plugins package -->
-    <gazebo reference="${name}">
+    <gazebo reference="${lidar_link}">
+      <xacro:if value="${gpu}">
+        <sensor type="gpu_ray" name="${name}-OS1-32">
+          <pose>0 0 0 0 0 0</pose>
+          <visualize>false</visualize>
+          <update_rate>${hz}</update_rate>
+          <ray>
+            <scan>
+              <horizontal>
+                <samples>${samples}</samples>
+                <resolution>1</resolution>
+                <min_angle>${min_angle}</min_angle>
+                <max_angle>${max_angle}</max_angle>
+              </horizontal>
+              <vertical>
+                <samples>32</samples>
+                <resolution>1</resolution>
+                <min_angle>${vfov_min}</min_angle>
+                <max_angle>${vfov_max}</max_angle>
+              </vertical>
+            </scan>
+            <range>
+              <min>${min_range}</min>
+              <max>${max_range}</max>
+              <resolution>0.03</resolution>
+            </range>
+          </ray>
+          <plugin name="gazebo_ros_laser_controller" filename="libgazebo_ros_ouster_gpu_laser.so">
+            <topicName>${topic_points}</topicName>
+            <frameName>${lidar_link}</frameName>
+            <min_range>${min_range}</min_range>
+            <max_range>${max_range}</max_range>
+            <gaussianNoise>${noise}</gaussianNoise>
+          </plugin>
+        </sensor>
+      </xacro:if>
+      <xacro:unless value="${gpu}">
         <sensor type="ray" name="${name}-OS1-32">
           <pose>0 0 0 0 0 0</pose>
@@ -77,4 +113,5 @@
           </plugin>
         </sensor>
+      </xacro:unless>
     </gazebo>
     <!-- IMU -->

File: arti_gazebo_ouster/urdf/OS1-64.urdf.xacro (robot description, xacro)
@@ -2,5 +2,5 @@
 <robot xmlns:xacro="http://ros.org/wiki/xacro" name="OS1-64">
   <xacro:property name="M_PI" value="3.1415926535897931" />
-  <xacro:macro name="OS1-64" params="*origin parent:=base_link name:=os1_sensor topic_points:=/os1_cloud_node/points topic_imu:=/os1_cloud_node/imu hz:=10 samples:=512 min_range:=0.9 max_range:=75.0 noise:=0.008 min_angle:=-${M_PI} max_angle:=${M_PI} lidar_link:=os1_lidar imu_link:=os1_imu vfov_min:=-.26 vfov_max:=.26">
+  <xacro:macro name="OS1-64" params="*origin parent:=base_link name:=os1_sensor topic_points:=/os1_cloud_node/points topic_imu:=/os1_cloud_node/imu hz:=10 samples:=512 min_range:=0.9 max_range:=75.0 noise:=0.008 min_angle:=-${M_PI} max_angle:=${M_PI} lidar_link:=os1_lidar imu_link:=os1_imu vfov_min:=-.26 vfov_max:=.26 gpu:=false">
     <joint name="${name}_mount_joint" type="fixed">
       <xacro:insert_block name="origin" />
@@ -22,5 +22,5 @@
       </collision>
       <visual name="base_visual">
-         <origin xyz="0 0 0.0" rpy="0 0 1.5707" />
+         <origin xyz="0 0 0.0365" rpy="0 0 1.5707" />
          <geometry>
 	         <mesh filename="package://arti_gazebo_ouster/meshes/os1_64.dae" />
@@ -43,5 +43,41 @@
     </joint>
     <!-- Gazebo requires the ouster_gazebo_plugins package -->
-    <gazebo reference="${name}">
+    <gazebo reference="${lidar_link}">
+      <xacro:if value="${gpu}">
+        <sensor type="gpu_ray" name="${name}-OS1-64">
+          <pose>0 0 0 0 0 0</pose>
+          <visualize>false</visualize>
+          <update_rate>${hz}</update_rate>
+          <ray>
+            <scan>
+              <horizontal>
+                <samples>${samples}</samples>
+                <resolution>1</resolution>
+                <min_angle>${min_angle}</min_angle>
+                <max_angle>${max_angle}</max_angle>
+              </horizontal>
+              <vertical>
+                <samples>64</samples>
+                <resolution>1</resolution>
+                <min_angle>${vfov_min}</min_angle>
+                <max_angle>${vfov_max}</max_angle>
+              </vertical>
+            </scan>
+            <range>
+              <min>${min_range}</min>
+              <max>${max_range}</max>
+              <resolution>0.03</resolution>
+            </range>
+          </ray>
+          <plugin name="gazebo_ros_laser_controller" filename="libgazebo_ros_ouster_gpu_laser.so">
+            <topicName>${topic_points}</topicName>
+            <frameName>${lidar_link}</frameName>
+            <min_range>${min_range}</min_range>
+            <max_range>${max_range}</max_range>
+            <gaussianNoise>${noise}</gaussianNoise>
+          </plugin>
+        </sensor>
+      </xacro:if>
+      <xacro:unless value="${gpu}">
         <sensor type="ray" name="${name}-OS1-64">
           <pose>0 0 0 0 0 0</pose>
@@ -77,4 +113,5 @@
           </plugin>
         </sensor>
+      </xacro:unless>
     </gazebo>
     <!-- IMU -->
